File: interface.kicad_sch (KiCad schematic)
At the start: 10 parts, among them J4 Conn_01x04_Pin, J5 Conn_01x05_Pin, Q2 BC817, Q3 BC817

Commit message: Fixed the Footprint assignment nonsense
Parts:
- C19, C20: footprint Resistor_SMD:R_0805_2012Metric -> Capacitor_SMD:C_0805_2012Metric
- J4: footprint Resistor_SMD:R_0805_2012Metric -> Connector_PinHeader_2.54mm:PinHeader_1x04_P2.54mm_Vertical
- J5: footprint Resistor_SMD:R_0805_2012Metric -> Connector_PinHeader_2.54mm:PinHeader_1x05_P2.54mm_Vertical
- Q2, Q3: footprint Resistor_SMD:R_0805_2012Metric -> Package_TO_SOT_SMD:SOT-23
Changed lines of the file:
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@@
 			)
 		)
-		(property "Footprint" "Resistor_SMD:R_0805_2012Metric"
+		(property "Footprint" "Connector_PinHeader_2.54mm:PinHeader_1x05_P2.54mm_Vertical"
 			(at 55.88 114.3 0)
 			(effects
@@
 			)
 		)
-		(property "Footprint" "Resistor_SMD:R_0805_2012Metric"
+		(property "Footprint" "Capacitor_SMD:C_0805_2012Metric"
 			(at 150.8252 71.12 0)
 			(effects
@@
 			)
 		)
-		(property "Footprint" "Resistor_SMD:R_0805_2012Metric"
+		(property "Footprint" "Connector_PinHeader_2.54mm:PinHeader_1x04_P2.54mm_Vertical"
 			(at 53.34 50.8 0)
 			(effects
@@
 			)
 		)
-		(property "Footprint" "Resistor_SMD:R_0805_2012Metric"
+		(property "Footprint" "Package_TO_SOT_SMD:SOT-23"
 			(at 185.42 128.905 0)
 			(effects
@@
 			)
 		)
-		(property "Footprint" "Resistor_SMD:R_0805_2012Metric"
+		(property "Footprint" "Capacitor_SMD:C_0805_2012Metric"
 			(at 211.7852 71.12 0)
 			(effects
@@
 			)
 		)
-		(property "Footprint" "Resistor_SMD:R_0805_2012Metric"
+		(property "Footprint" "Package_TO_SOT_SMD:SOT-23"
 			(at 185.42 103.505 0)
 			(effects

Commit message: Power copper zones and Placement complete
Changed lines of the file:
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@@
-		)
-	)
-	(label "+3.3V"
-		(at 45.72 99.06 180)
-		(effects
-			(font
-				(size 1.27 1.27)
-			)
-			(justify right bottom)
-		)
-	)
-	(label "+3.3V"
-		(at 45.72 38.1 180)
-		(effects
-			(font
-				(size 1.27 1.27)
-			)
-			(justify right bottom)
 		)
 	)
@@
 	)
 	(symbol
+		(lib_id "power:+3.3V")
+		(at 45.72 99.06 0)
+		(unit 1)
+		(exclude_from_sim no)
+		(in_bom yes)
+		(on_board yes)
+		(dnp no)
+		(fields_autoplaced yes)
+		(property "Reference" "#PWR049"
+			(at 45.72 102.87 0)
+			(effects
+				(font
+					(size 1.27 1.27)
+				)
+				(hide yes)
+			)
+		)
+		(property "Value" "+3.3V"
+			(at 45.72 93.98 0)
+			(effects
+				(font
+					(size 1.27 1.27)
+				)
+			)
+		)
+		(property "Footprint" ""
+			(at 45.72 99.06 0)
+			(effects
+				(font
+					(size 1.27 1.27)
+				)
+				(hide yes)
+			)
+		)
+		(property "Datasheet" ""
+			(at 45.72 99.06 0)
+			(effects
+				(font
+					(size 1.27 1.27)
+				)
+				(hide yes)
+			)
+		)
+		(property "Description" "Power symbol creates a global label with name \"+3.3V\""
+			(at 45.72 99.06 0)
+			(effects
+				(font
+					(size 1.27 1.27)
+				)
+				(hide yes)
+			)
+		)
+		(pin "1"
+		)
+		(instances
+			(project ""
+				(path "/8e18a6b6-2497-40ab-aacd-16656297d80d/0980fd62-4755-455b-bc26-b8079d26a0ec/5cb12f4a-c7bb-4896-9e22-73783dfb5b5b"
+					(reference "#PWR049")
+					(unit 1)
+				)
+			)
+		)
+	)
+	(symbol
 		(lib_id "Device:R")
 		(at 158.75 101.6 90)
@@
 					(unit 1)
 				)
+			)
+		)
+	)
+	(symbol
+		(lib_id "power:+3.3V")
+		(at 45.72 38.1 0)
+		(unit 1)
+		(exclude_from_sim no)
+		(in_bom yes)
+		(on_board yes)
+		(dnp no)
+		(fields_autoplaced yes)
+		(property "Reference" "#PWR048"
+			(at 45.72 41.91 0)
+			(effects
+				(font
+					(size 1.27 1.27)
+				)
+				(hide yes)
+			)
+		)
+		(property "Value" "+3.3V"
+			(at 45.72 33.02 0)
+			(effects
+				(font
+					(size 1.27 1.27)
+				)
+			)
+		)
+		(property "Footprint" ""
+			(at 45.72 38.1 0)
+			(effects
+				(font
+					(size 1.27 1.27)
+				)
+				(hide yes)
+			)
+		)
+		(property "Datasheet" ""
+			(at 45.72 38.1 0)
+			(effects
+				(font
+					(size 1.27 1.27)
+				)
+				(hide yes)
+			)
+		)
+		(property "Description" "Power symbol creates a global label with name \"+3.3V\""
+			(at 45.72 38.1 0)
+			(effects
+				(font
+					(size 1.27 1.27)
+				)
+				(hide yes)
+			)
+		)
+		(pin "1"
+		)
+		(instances
+			(project ""
+				(path "/8e18a6b6-2497-40ab-aacd-16656297d80d/0980fd62-4755-455b-bc26-b8079d26a0ec/5cb12f4a-c7bb-4896-9e22-73783dfb5b5b"
+					(reference "#PWR048")
+					(unit 1)
+				)

Commit message: Completed layout fix
Parts:
- S1, S2: symbol USLPT2819DT2TR:USLPT2819DT2TR -> dk_Tactile-Switches:TL3315NF160Q; Category (none) -> Switches; DK_Datasheet_Link (none) -> http://spec_sheets.e-switch.com/specs/P010337.pdf; DK_Detail_Page (none) -> /product-detail/en/e-switch/TL3315NF160Q/EG4621CT-ND/1870401; Description_1 Tactile Switch SPST-NO Top Actuated Surface Mount -> SWITCH TACTILE SPST-NO 0.05A 15V; Digi-Key_PN (none) -> EG4621CT-ND; Family (none) -> Tactile Switches; MPN (none) -> TL3315NF160Q; Manufacturer (none) -> E-Switch; Status (none) -> Active
Connections:
- net BOOT: now also Q3.3 (C), S1.2; no longer Q3.2 (E), S1.3
- net DTR: now also Q3.2 (E); no longer Q3.3 (C)
- net EN: now also S2.2; no longer S2.3
- net GND: now also S1.3, S2.3; no longer S1.2, S2.2
