File: sensors.kicad_sch (KiCad schematic)
At the start: 19 parts, among them Q4 TEMT6000X01, U6 MAX4466EXK, U7 BME280

Commit message: Completed layout fix
Parts:
- added C23, C24: 10nF, Capacitor_SMD:C_0805_2012Metric, symbol Device:C
- added C25: 0.1uF, Capacitor_SMD:C_0805_2012Metric, symbol Device:C
- added R32: 35WR100KLFTR, 35WR100KLFTR:TRIM_35WR100KLFTR, symbol 35WR100KLFTR:35WR100KLFTR
- C21: value 1uF -> 10uF
- R24: value 100k -> 22k
- R25: value 10k -> 1k
Connections:
- net +3.3V: now also Q4.3, C25.1; no longer R23.1
- net GND: now also R23.2, C23.2, C24.2, C25.2; no longer Q4.1
- net MIC_OUT: now also R32.1, R32.2; no longer R24.1
- net PHOTO_C: now also Q4.1, R23.1, C23.1, C24.1; no longer Q4.3, R23.2
- new net: R24.1, R32.3
Other:
- moved on the sheet: C17, Q4, R23, R24
