File: _autosave-ESP32_CustomBoard.kicad_pcb (KiCad board)
At the start: 4 copper layers, 84.5 x 57.2 mm, 84 parts, among them J1 SS-52400-003, J2 B2B-PH-SM4-TB, J3 GSD090012SEU, J4 Conn_01x04_Pin, J5 Conn_01x05_Pin, Q2 BC817, Q3 BC817, Q4 TEMT6000X01, U1 MCP73871, U2 CP2102N-Axx-xQFN20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

Commit message: Power copper zones and Placement complete
Parts:
- moved C3 36.1 mm to (153.3, 107.2)
- moved C5 36.1 mm to (156.0, 107.2)
- moved C8 36.1 mm to (158.5, 107.8)
- moved C7 36.1 mm to (150.6, 113.7)
- moved VR1 36.1 mm to (155.7, 114.0)
- moved J2 19.7 mm to (172.0, 114.1)
- moved D2 19.6 mm to (187.8, 117.1)
- moved D3 19.6 mm to (192.2, 117.1)
- moved LED3 19.6 mm to (183.4, 117.4)
- moved R1 19.6 mm to (192.0, 112.5)
- moved R3 19.6 mm to (184.9, 110.8)
- moved R6 19.6 mm to (189.8, 117.3)
- moved R7 19.6 mm to (194.1, 117.3)
- moved R4 19.6 mm to (195.9, 109.6)
- moved R5 19.6 mm to (195.9, 107.5)
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Connections:
- C10 pad 2: /ESP32_module/+3.3V -> +3.3V
- C11 pad 1: /ESP32_module/+3.3V -> +3.3V
- C12 pad 1: /ESP32_module/+3.3V -> +3.3V
- C13 pad 1: /ESP32_module/+3.3V -> +3.3V
- C14 pad 1: /ESP32_module/+3.3V -> +3.3V
- C15 pad 1: /ESP32_module/Sensors/+3.3V -> +3.3V
- C16 pad 1: /ESP32_module/Sensors/+3.3V -> +3.3V
- C5 pad 1: /+3.3V -> +3.3V
- C6 pad 2: /ESP32_module/+3.3V -> +3.3V
- C8 pad 1: /+3.3V -> +3.3V
- C9 pad 2: /ESP32_module/+3.3V -> +3.3V
- J3 pad 4: /ESP32_module/+3.3V -> +3.3V
- J4 pad 4: /ESP32_module/User Interface/+3.3V -> +3.3V
- J5 pad 5: /ESP32_module/User Interface/+3.3V -> +3.3V
- LED1 pad 2: /+3.3V -> +3.3V
- R11 pad 1: /ESP32_module/+3.3V -> +3.3V
- R12 pad 1: /ESP32_module/+3.3V -> +3.3V
- R13 pad 1: /ESP32_module/+3.3V -> +3.3V
- R19 pad 2: /ESP32_module/+3.3V -> +3.3V
- R21 pad 1: /ESP32_module/Sensors/+3.3V -> +3.3V
- R22 pad 1: /ESP32_module/Sensors/+3.3V -> +3.3V
- R23 pad 1: /ESP32_module/Sensors/+3.3V -> +3.3V
- R26 pad 1: /ESP32_module/Sensors/+3.3V -> +3.3V
- R28 pad 1: /ESP32_module/Sensors/+3.3V -> +3.3V
- U2 pad 6: /ESP32_module/+3.3V -> +3.3V
- U2 pad 7: /ESP32_module/+3.3V -> +3.3V
- U4 pad 3: /ESP32_module/+3.3V -> +3.3V
- U4 pad 7: /ESP32_module/+3.3V -> +3.3V
- U4 pad 8: /ESP32_module/+3.3V -> +3.3V
- U5 pad 1: /ESP32_module/+3.3V -> +3.3V
- U6 pad 5: /ESP32_module/Sensors/+3.3V -> +3.3V
- U7 pad 2: /ESP32_module/Sensors/+3.3V -> +3.3V
- U7 pad 6: /ESP32_module/Sensors/+3.3V -> +3.3V
- U7 pad 8: /ESP32_module/Sensors/+3.3V -> +3.3V
- VR1 pad 2: /+3.3V -> +3.3V
Routing:
- net /USB_DP: track 0.00 -> 19.9 mm
- net /USB_DN: track 0.00 -> 19.9 mm
- added copper zone on In2.Cu, net +3.3V
- added copper zone on In2.Cu, net /+5V_USB
- added copper zone on In1.Cu, net GND
- removed copper zone on In2.Cu, net GND
