File: _autosave-ESP32_CustomBoard.kicad_pcb (KiCad board)
At the start: 4 copper layers, 84.5 x 57.2 mm, 84 parts, among them J1 SS-52400-003, J2 B2B-PH-SM4-TB, J3 GSD090012SEU, J4 Conn_01x04_Pin, J5 Conn_01x05_Pin, Q2 BC817, Q3 BC817, Q4 TEMT6000X01, U1 MCP73871, U2 CP2102N-Axx-xQFN20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

Commit message: fixed errors, completed silkscreen and 3D assignment
Parts:
- moved C10 0.91 mm to (208.2, 72.3)
Changed lines of the file:
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@@
 		)
 		(fp_circle
-			(center -10.5 -2.9)
-			(end -10.4 -2.9)
+			(center -10.5 -3.93)
+			(end -10.4 -3.93)
 			(stroke
 				(width 0.2)
@@
 		)
 		(fp_circle
-			(center -10.5 -2.9)
-			(end -10.4 -2.9)
+			(center -10.5 -3.93)
+			(end -10.4 -3.93)
 			(stroke
 				(width 0.2)
@@
 	(footprint "Capacitor_SMD:C_0805_2012Metric"
 		(layer "F.Cu")
-		(at 208.18 73.23)
+		(at 208.21 72.32)
 		(descr "Capacitor SMD 0805 (2012 Metric), square (rectangular) end terminal, IPC-7351 nominal, (Body size source: IPC-SM-782 page 76, https://www.pcb-3d.com/wordpress/wp-content/uploads/ipc-sm-782a_amendment_1_and_2.pdf, https://docs.google.com/spreadsheets/d/1BsfQQcO9C6DZCsRaXUlFlo91Tg2WpOkGARC1WS5S8t0/edit?usp=sharing), generated with kicad-footprint-generator")
 		(tags "capacitor")
@@
 	)
 	(gr_text "GPIO19"
-		(at 182.542838 70.106667 90)
+		(at 182.542838 70.436666 90)
 		(layer "F.SilkS")
 		(effects
@@
 	)
 	(gr_text "+3.3V"
-		(at 174.922838 69.440001 90)
+		(at 174.922838 69.77 90)
 		(layer "F.SilkS")
 		(effects
@@
 	)
 	(gr_text "GPIO18"
-		(at 180.002838 70.106667 90)
+		(at 180.002838 70.436666 90)
 		(layer "F.SilkS")
 		(effects
@@
 	)
 	(gr_text "GPIO8\n"
-		(at 177.462838 69.44 90)
+		(at 177.462838 69.769999 90)
 		(layer "F.SilkS")
 		(effects
@@
 	)
 	(segment
+		(start 207.1204 72.1804)
+		(end 207.26 72.32)
+		(width 0.5)
+		(layer "F.Cu")
+		(net 1)
+	)
+	(segment
 		(start 158.2548 96.45)
 		(end 159.4538 96.45)
@@
 	)
 	(segment
+		(start 205.010806 72.1804)
+		(end 207.1204 72.1804)
+		(width 0.5)
+		(layer "F.Cu")
+		(net 1)
+	)
+	(segment
 		(start 177.6675 92.1258)
 		(end 177.005001 92.1258)
@@
 	)
 	(segment
-		(start 205.010806 72.1804)
-		(end 206.1804 72.1804)
-		(width 0.5)
-		(layer "F.Cu")
-		(net 1)
-	)
-	(segment
 		(start 164.3615 90.5275)
 		(end 165.2524 89.6366)
@@
 	)
 	(segment
-		(start 206.1804 72.1804)
-		(end 207.23 73.23)
-		(width 0.5)
-		(layer "F.Cu")
-		(net 1)
-	)
-	(segment
 		(start 157.8845 101.473)
 		(end 157.8845 98.6997)
@@
 	)
 	(segment
-		(start 209.13 73.23)
-		(end 210.4316 71.9284)
-		(width 0.5)
-		(layer "F.Cu")
-		(net 5)
-	)
-	(segment
 		(start 181.35467 73.7209)
 		(end 179.6182 73.7209)
@@
 	)
 	(segment
+		(start 211.1685 71.9284)
+		(end 209.5516 71.9284)
+		(width 0.5)
+		(layer "F.Cu")
+		(net 5)
+	)
+	(segment
 		(start 181.0052 74.9239)
 		(end 181.25767 74.9239)
@@
 	)
 	(segment
-		(start 210.4316 71.9284)
-		(end 211.1685 71.9284)
-		(width 0.5)
-		(layer "F.Cu")
-		(net 5)
-	)
-	(segment
 		(start 182.2094 93.1932)
 		(end 181.9094 92.8932)
@@
 		(width 0.5)
 		(layer "F.Cu")
+		(net 5)
+	)
+	(segment
+		(start 209.5516 71.9284)
+		(end 209.16 72.32)
+		(width 0.5)
+		(layer "F.Cu")
