File: ESP32_CustomBoard.kicad_pcb (KiCad board)
At the start: 4 copper layers, 84.5 x 57.2 mm, 84 parts, among them J1 SS-52400-003, J2 B2B-PH-SM4-TB, J3 GSD090012SEU, J4 Conn_01x04_Pin, J5 Conn_01x05_Pin, Q2 BC817, Q3 BC817, Q4 TEMT6000X01, U1 MCP73871, U2 CP2102N-Axx-xQFN20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

Commit message: Completed Routing
Parts:
- moved TP4 46.6 mm to (231.1, 71.9)
- moved TP3 37.8 mm to (204.4, 80.4)
- moved C3 36.1 mm to (153.3, 107.2)
- moved C5 36.1 mm to (156.0, 107.2)
- moved C8 36.1 mm to (158.5, 107.8)
- moved C7 36.1 mm to (150.6, 113.7)
- moved VR1 36.1 mm to (155.7, 114.0)
- moved TP1 29.5 mm to (208.2, 85.6)
- moved TP5 28.5 mm to (228.7, 86.7)
- moved TP2 24.0 mm to (201.5, 91.3)
- moved J2 19.7 mm to (172.0, 114.1)
- moved LED3 19.6 mm to (183.4, 116.1)
- moved D2 19.6 mm to (187.8, 116.4)
- moved D3 19.6 mm to (192.2, 117.1)
- moved R1 19.6 mm to (192.0, 112.5)
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Connections:
- C10 pad 2: /ESP32_module/+3.3V -> +3.3V
- C11 pad 1: /ESP32_module/+3.3V -> +3.3V
- C12 pad 1: /ESP32_module/+3.3V -> +3.3V
- C13 pad 1: /ESP32_module/+3.3V -> +3.3V
- C14 pad 1: /ESP32_module/+3.3V -> +3.3V
- C15 pad 1: /ESP32_module/Sensors/+3.3V -> +3.3V
- C16 pad 1: /ESP32_module/Sensors/+3.3V -> +3.3V
- C5 pad 1: /+3.3V -> +3.3V
- C6 pad 2: /ESP32_module/+3.3V -> +3.3V
- C8 pad 1: /+3.3V -> +3.3V
- C9 pad 2: /ESP32_module/+3.3V -> +3.3V
- J3 pad 4: /ESP32_module/+3.3V -> +3.3V
- J4 pad 4: /ESP32_module/User Interface/+3.3V -> +3.3V
- J5 pad 5: /ESP32_module/User Interface/+3.3V -> +3.3V
- LED1 pad 2: /+3.3V -> +3.3V
- R11 pad 1: /ESP32_module/+3.3V -> +3.3V
- R12 pad 1: /ESP32_module/+3.3V -> +3.3V
- R13 pad 1: /ESP32_module/+3.3V -> +3.3V
- R19 pad 2: /ESP32_module/+3.3V -> +3.3V
- R21 pad 1: /ESP32_module/Sensors/+3.3V -> +3.3V
- R22 pad 1: /ESP32_module/Sensors/+3.3V -> +3.3V
- R23 pad 1: /ESP32_module/Sensors/+3.3V -> +3.3V
- R26 pad 1: /ESP32_module/Sensors/+3.3V -> +3.3V
- R28 pad 1: /ESP32_module/Sensors/+3.3V -> +3.3V
- U2 pad 4: Net-(U2-D+) -> /ESP32_module/USB_P
- U2 pad 5: Net-(U2-D-) -> /ESP32_module/USB_N
- U2 pad 6: /ESP32_module/+3.3V -> +3.3V
- U2 pad 7: /ESP32_module/+3.3V -> +3.3V
- U3 pad 1: Net-(U2-D+) -> /ESP32_module/USB_N
- U3 pad 2: /VBUS -> GND
- U3 pad 3: Net-(U2-D-) -> /ESP32_module/USB_P
- U3 pad 4: /USB_DN -> /USB_DP
- U3 pad 5: GND -> /VBUS
- U3 pad 6: /USB_DP -> /USB_DN
- U4 pad 3: /ESP32_module/+3.3V -> +3.3V
- U4 pad 7: /ESP32_module/+3.3V -> +3.3V
- U4 pad 8: /ESP32_module/+3.3V -> +3.3V
- U5 pad 1: /ESP32_module/+3.3V -> +3.3V
- U6 pad 5: /ESP32_module/Sensors/+3.3V -> +3.3V
- U7 pad 2: /ESP32_module/Sensors/+3.3V -> +3.3V
- U7 pad 6: /ESP32_module/Sensors/+3.3V -> +3.3V
- U7 pad 8: /ESP32_module/Sensors/+3.3V -> +3.3V
- VR1 pad 2: /+3.3V -> +3.3V
Routing:
- net GND: track 0.00 -> 268.4 mm, vias 0 -> 23
- net +3.3V: track 0.00 -> 148.1 mm, vias 0 -> 10
- net /ESP32_module/PHOTO_C: track 0.00 -> 84.2 mm, vias 0 -> 2
- net /ESP32_module/MISO_DO: track 0.00 -> 74.7 mm, vias 0 -> 2
- net /ESP32_module/SCL: track 0.00 -> 66.3 mm, vias 0 -> 1
- net /ESP32_module/GPIO18: track 0.00 -> 57.9 mm, vias 0 -> 1
- net /ESP32_module/GPIO19: track 0.00 -> 55.3 mm, vias 0 -> 1
- net /ESP32_module/MIC_OUT: track 0.00 -> 53.9 mm, vias 0 -> 2
- net /ESP32_module/RX_TX: track 0.00 -> 52.1 mm, vias 0 -> 2
- net /ESP32_module/TX_RX: track 0.00 -> 51.5 mm, vias 0 -> 2
- net /ESP32_module/GPIO8: track 0.00 -> 49.7 mm, vias 0 -> 1
- net /+5V: track 0.00 -> 48.9 mm, vias 0 -> 2
- net /ESP32_module/SDA: track 0.00 -> 45.1 mm
- net /+5V_USB: track 0.00 -> 43.8 mm, vias 0 -> 4
- net /ESP32_module/CS: track 0.00 -> 42.8 mm, vias 0 -> 2
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- added copper zone on In2.Cu, net +3.3V
- added copper zone on In2.Cu, net /+5V_USB
- added copper zone on In2.Cu, net /VBUS
- added copper zone on In1.Cu, net GND
- removed copper zone on In2.Cu, net GND
