File: ESP32_CustomBoard.kicad_pcb (KiCad board)
At the start: 4 copper layers, 84.5 x 57.2 mm, 84 parts, among them J1 SS-52400-003, J2 B2B-PH-SM4-TB, J3 GSD090012SEU, J4 Conn_01x04_Pin, J5 Conn_01x05_Pin, Q2 BC817, Q3 BC817, Q4 TEMT6000X01, U1 MCP73871, U2 CP2102N-Axx-xQFN20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

Commit message: Schematic Fixes
Parts:
- moved C10 0.91 mm to (208.2, 72.3)
Routing:
- net +3.3V: track 151.6 -> 149.5 mm, vias 10 -> 13
- net GND: track 290.8 -> 291.7 mm
Changed lines of the file:
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@@
 			(plot_on_all_layers_selection 0x00000000_00000000_00000000_00000000)
 			(disableapertmacros no)
-			(usegerberextensions no)
+			(usegerberextensions yes)
 			(usegerberattributes yes)
 			(usegerberadvancedattributes yes)
@@
 			(outputformat 1)
 			(mirror no)
-			(drillshape 1)
+			(drillshape 0)
 			(scaleselection 1)
-			(outputdirectory "")
+			(outputdirectory "GERBERS/")
 		)
 	)
@@
 		)
 		(fp_circle
-			(center -10.5 -2.9)
-			(end -10.4 -2.9)
+			(center -10.5 -3.93)
+			(end -10.4 -3.93)
 			(stroke
 				(width 0.2)
@@
 		)
 		(fp_circle
-			(center -10.5 -2.9)
-			(end -10.4 -2.9)
+			(center -10.5 -3.93)
+			(end -10.4 -3.93)
 			(stroke
 				(width 0.2)
@@
 	(footprint "Capacitor_SMD:C_0805_2012Metric"
 		(layer "F.Cu")
-		(at 208.18 73.23)
+		(at 208.21 72.32)
 		(descr "Capacitor SMD 0805 (2012 Metric), square (rectangular) end terminal, IPC-7351 nominal, (Body size source: IPC-SM-782 page 76, https://www.pcb-3d.com/wordpress/wp-content/uploads/ipc-sm-782a_amendment_1_and_2.pdf, https://docs.google.com/spreadsheets/d/1BsfQQcO9C6DZCsRaXUlFlo91Tg2WpOkGARC1WS5S8t0/edit?usp=sharing), generated with kicad-footprint-generator")
 		(tags "capacitor")
@@
 	)
 	(gr_text "GPIO19"
-		(at 182.542838 70.106667 90)
+		(at 182.542838 70.436666 90)
 		(layer "F.SilkS")
 		(effects
@@
 	)
 	(gr_text "+3.3V"
-		(at 174.922838 69.440001 90)
+		(at 174.922838 69.77 90)
 		(layer "F.SilkS")
 		(effects
@@
 	)
 	(gr_text "GPIO18"
-		(at 180.002838 70.106667 90)
+		(at 180.002838 70.436666 90)
 		(layer "F.SilkS")
 		(effects
@@
 	)
 	(gr_text "GPIO8\n"
-		(at 177.462838 69.44 90)
+		(at 177.462838 69.769999 90)
 		(layer "F.SilkS")
 		(effects
@@
 	)
 	(segment
+		(start 181.0052 73.0052)
+		(end 181 73)
+		(width 0.254)
+		(layer "F.Cu")
+		(net 1)
+	)
+	(segment
 		(start 159.9746 71.9658)
 		(end 158.1404 73.8)
@@
 	)
 	(segment
+		(start 207.1204 72.1804)
+		(end 207.26 72.32)
+		(width 0.5)
+		(layer "F.Cu")
+		(net 1)
+	)
+	(segment
 		(start 158.2548 96.45)
 		(end 159.4538 96.45)
@@
 	)
 	(segment
+		(start 205.010806 72.1804)
+		(end 207.1204 72.1804)
+		(width 0.5)
+		(layer "F.Cu")
+		(net 1)
+	)
+	(segment
 		(start 177.6675 92.1258)
 		(end 177.005001 92.1258)
@@
 	)
 	(segment
-		(start 205.010806 72.1804)
-		(end 206.1804 72.1804)
-		(width 0.5)
-		(layer "F.Cu")
-		(net 1)
-	)
-	(segment
 		(start 164.3615 90.5275)
 		(end 165.2524 89.6366)
@@
 	)
 	(segment
+		(start 181.0052 74.2739)
+		(end 181.0052 73.0052)
+		(width 0.254)
+		(layer "F.Cu")
+		(net 1)
+	)
+	(segment
 		(start 175.6562 75.692)
 		(end 172.4584 72.4942)
@@
 	)
 	(segment
-		(start 206.1804 72.1804)
-		(end 207.23 73.23)
-		(width 0.5)
-		(layer "F.Cu")
-		(net 1)
-	)
-	(segment
 		(start 157.8845 101.473)
 		(end 157.8845 98.6997)
@@
 	)
 	(via
-		(at 166.4716 94.361)
+		(at 181 73)
 		(size 0.6)
 		(drill 0.4)
@@
 	)
 	(via
-		(at 165.2524 89.6366)
+		(at 166.4716 94.361)
 		(size 0.6)
 		(drill 0.4)
@@
 	)
 	(via
-		(at 188.4172 74.7268)
+		(at 165.2524 89.6366)
 		(size 0.6)
 		(drill 0.4)
@@
 	)
 	(via
-		(at 179.832 75.184)
+		(at 188.4172 74.7268)
 		(size 0.6)
 		(drill 0.4)
@@
 	)
 	(segment
-		(start 179.6182 73.7209)
-		(end 179.0652 74.2739)
-		(width 0.254)
-		(layer "F.Cu")
-		(net 5)
-	)
-	(segment
 		(start 178.2493 74.2739)
 		(end 177.5562 74.967)
@@
 	)
 	(segment
-		(start 181.5782 73.94443)
-		(end 181.35467 73.7209)
-		(width 0.254)
-		(layer "F.Cu")
-		(net 5)
-	)
-	(segment
 		(start 167.3925 67.0926)
 		(end 167.3925 70.2971)
@@
 	)
 	(segment
+		(start 181.0052 74.9239)
+		(end 182.2161 74.9239)
+		(width 0.3)
+		(layer "F.Cu")
+		(net 5)
+	)
+	(segment
 		(start 228.6 90.8)
 		(end 227.190273 89.390273)
@@
 	)
 	(segment
-		(start 181.25767 74.9239)
-		(end 181.5782 74.60337)
-		(width 0.254)
-		(layer "F.Cu")
-		(net 5)
-	)
-	(segment
 		(start 179.008967 88.813567)
 		(end 179.008967 87.5382)
@@
 	)
 	(segment
-		(start 209.13 73.23)
-		(end 210.4316 71.9284)
-		(width 0.5)
-		(layer "F.Cu")
-		(net 5)
-	)
-	(segment
-		(start 181.35467 73.7209)
-		(end 179.6182 73.7209)
-		(width 0.254)
-		(layer "F.Cu")
-		(net 5)
-	)
-	(segment
 		(start 169.4742 70.5942)
 		(end 167.5246 70.5942)
@@
 	)
 	(segment
-		(start 181.0052 74.9239)
-		(end 181.25767 74.9239)
-		(width 0.254)
+		(start 211.1685 71.9284)
+		(end 209.5516 71.9284)
+		(width 0.5)
 		(layer "F.Cu")
 		(net 5)
@@
 	)
 	(segment
-		(start 210.4316 71.9284)
-		(end 211.1685 71.9284)
-		(width 0.5)
-		(layer "F.Cu")
-		(net 5)
-	)
-	(segment
 		(start 182.2094 93.1932)
 		(end 181.9094 92.8932)
@@
 	)
 	(segment
+		(start 182.2161 74.9239)
+		(end 182.22 74.92)
+		(width 0.3)
+		(layer "F.Cu")
+		(net 5)
+	)
+	(segment
 		(start 189.7769 90.4005)
 		(end 190.4492 89.7282)
@@
 	)
 	(segment
+		(start 209.5516 71.9284)
+		(end 209.16 72.32)
+		(width 0.5)
+		(layer "F.Cu")
+		(net 5)
+	)
+	(segment
 		(start 176.2506 87.5382)
 		(end 179.008967 87.5382)
@@
 	)
 	(segment
+		(start 179.0652 73.0348)
+		(end 179.07 73.03)
+		(width 0.254)
+		(layer "F.Cu")
+		(net 5)
+	)
+	(segment
 		(start 148.2742 81.7482)
 		(end 150.2156 79.8068)
@@
 	)
 	(segment
-		(start 181.5782 74.60337)
-		(end 181.5782 73.94443)
+		(start 179.0652 74.2739)
+		(end 179.0652 73.0348)
 		(width 0.254)
 		(layer "F.Cu")
@@
 	)
 	(via
+		(at 179.07 73.03)
+		(size 0.6)
+		(drill 0.4)
+		(layers "F.Cu" "B.Cu")
+		(net 5)
+	)
+	(via
 		(at 155.7274 79.0448)
 		(size 0.6)
@@
 		(size 0.6)
 		(drill 0.4)
+		(layers "F.Cu" "B.Cu")
+		(net 5)
+	)
+	(via
+		(at 182.22 74.92)
+		(size 0.6)
+		(drill 0.4)
+		(layers "F.Cu" "B.Cu")
+		(net 5)
+	)
+	(via
+		(at 182.22 74.92)
+		(size 0.6)
+		(drill 0.4)

Commit message: Completed layout fix
Parts:
- added C23: 10nF, Capacitor_SMD:C_0805_2012Metric, F.Cu at (230.9, 74.5)
- added C24: 10nF, Capacitor_SMD:C_0805_2012Metric, F.Cu at (156.7, 82.0)
- added C25: 0.1uF, Capacitor_SMD:C_0805_2012Metric, F.Cu at (151.3, 82.0)
- added FB1: FBMJ2125HM330-TV, FBMJ2125HM330-TV:BEADC2012X105N, F.Cu at (186.1, 105.5)
- added R32: 35WR100KLFTR, 35WR100KLFTR:TRIM_35WR100KLFTR, F.Cu at (165.7, 78.0)
- C21: value 1uF -> 10uF
- R24: value 100k -> 22k
- R25: value 10k -> 1k
- TP4: moved to B.Cu
- moved TP4 16.6 mm to (215.8, 79.1)
- moved C17 5.33 mm to (161.2, 77.3), turned to -90 degrees
- moved S1 1.64 mm to (191.5, 70.4)
- moved Q3 1.61 mm to (190.6, 74.5)
- moved S2 1.60 mm to (198.2, 70.4)
- moved Q2 1.56 mm to (198.9, 74.5)
- moved C19 1.39 mm to (190.3, 78.0)
- moved C20 1.29 mm to (199.2, 78.0)
- moved R31 0.70 mm to (194.7, 76.8)
- moved R30 0.19 mm to (194.7, 74.5)
Connections:
- Q3 pad 2: /ESP32_module/BOOT -> /ESP32_module/DTR
- Q3 pad 3: /ESP32_module/DTR -> /ESP32_module/BOOT
- Q4 pad 1: GND -> /ESP32_module/PHOTO_C
- Q4 pad 3: /ESP32_module/PHOTO_C -> +3.3V
- R23 pad 1: +3.3V -> /ESP32_module/PHOTO_C
- R23 pad 2: /ESP32_module/PHOTO_C -> GND
- R24 pad 1: /ESP32_module/MIC_OUT -> Net-(R24-Pad1)
- S1 pad 2: GND -> /ESP32_module/BOOT
- S1 pad 3: /ESP32_module/BOOT -> GND
- S2 pad 2: GND -> /ESP32_module/EN
- S2 pad 3: /ESP32_module/EN -> GND
- U1 pad 1: /+5V -> Net-(FB1-Pad1)
- U1 pad 20: /+5V -> Net-(FB1-Pad1)
- U5 pad 18: /ESP32_module/CS_SD -> /ESP32_module/MIC_OUT
- U5 pad 4: /ESP32_module/MIC_OUT -> /ESP32_module/CS_SD
Routing:
- net /ESP32_module/CS_SD: track 2.30 -> 50.4 mm, vias 0 -> 2
- net /ESP32_module/MIC_OUT: track 53.9 -> 78.3 mm
- net /ESP32_module/MISO_DO: track 74.7 -> 56.6 mm
- net GND: track 291.7 -> 300.6 mm, vias 25 -> 28
- net /ESP32_module/PHOTO_C: track 84.2 -> 91.8 mm
- net /ESP32_module/DTR: track 22.0 -> 28.0 mm, vias 0 -> 2
- net /+5V_USB: track 46.0 -> 41.6 mm
- net Net-(U6-IN-): track 8.32 -> 12.4 mm
- net Net-(FB1-Pad1): track 0.00 -> 3.56 mm
- net /ESP32_module/BOOT: track 41.0 -> 37.9 mm
- net Net-(R24-Pad1): track 0.00 -> 2.67 mm
- net /ESP32_module/SCL: track 66.3 -> 63.8 mm
- net +3.3V: track 149.5 -> 146.9 mm, vias 13 -> 11
- net /ESP32_module/RTS: track 21.6 -> 22.7 mm
- net /ESP32_module/EN: track 32.8 -> 31.7 mm
- removed copper zone on F.Cu, net /+5V
Other:
- board size 84.5 x 57.2 mm -> 85 x 57.2 mm
