File: ESP32_CustomBoard.kicad_sch (KiCad schematic)
At the start: 0 parts

Commit message: Completed Sheet 2- ESP32 Module
Parts:
- added C1, C7: 0.1uF, symbol Device:C
- added C2, C8: 0..1uF, symbol Device:C
- added C3, C5: 10uF, symbol Device:C_Polarized
- added D2: LTST-C170TBKT, digikey-footprints:0805, symbol dk_LED-Indication-Discrete:LTST-C170TBKT
- added D3: LTST-C170GKT, LTST-C170GKT:LED_LTST-C170GKT, symbol LTST-C170GKT:LTST-C170GKT
- added F1: 0ZCH0110AF2E, 0ZCH0110AF2E:FUSC3225X100N, symbol 0ZCH0110AF2E:0ZCH0110AF2E
- added J1: SS-52400-003, SS-52400-003:BELFUSE_SS-52400-003, symbol SS-52400-003:SS-52400-003
- added J2: B2B-PH-SM4-TB, B2B-PH-SM4-TB:JST_B2B-PH-SM4-TB, symbol B2B-PH-SM4-TB:B2B-PH-SM4-TB
- added LED1, LED3: LTST-C170KRKT, LED_LTST-C170KRKT_LTO, symbol LTST-C170KRKT:LTST-C170KRKT
- added R1, R3: 10k, symbol Device:R
- added R10, R6, R7, R8: 470, symbol Device:R
- added R2, R9: 5.1k, symbol Device:R
- added R4: 20k, symbol Device:R
- added R5: 2k, symbol Device:R
- added U1: MCP73871, Package_DFN_QFN:QFN-20-1EP_4x4mm_P0.5mm_EP2.5x2.5mm, symbol Battery_Management:MCP73871
- added VR1: LM1117MPX-3.3, LM1117MPX-3.3:VREG_LM1117MPX-3.3, symbol LM1117MPX-3.3:LM1117MPX-3.3
Connections:
- new net: D2.1, R6.1
- new net: D2.2, U1.7 (STAT2)
- new net: R1.1, U1.9 (~{TE})
- new net: R5.2, U1.13 (PROG1)
- new net: J1.B5 (CC2), R2.2
- new net: J1.A5 (CC1), R9.1
- new net: LED3.2, R8.1
- new net: R4.2, U1.12 (PROG3)
- new net: R3.2, U1.5 (THERM)
- new net: LED3.1, U1.6 (~{PG})
- new net: D3.1, U1.8 (STAT1/~{LBO})
- new net: D3.2, R7.1
- new net +3.3V: C5.1, C8.1, LED1.2, VR1.2 (VOUT_2)
- new net +5V: C3.1, C7.1, U1.1 (OUT), U1.20 (OUT), VR1.3 (VIN)
- new net +5V_USB: C2.1, F1.1, R6.2, R7.2, R8.2, U1.17 (CE), U1.18 (IN), U1.19 (IN), U1.2 (VPCC), U1.4 (PROG2)
- new net GND: C1.2, C2.2, C3.2, C5.2, C7.2, C8.2, J1.A1 (GNDA1), J1.A12 (GNDA2), J1.B1 (GNDB1), J1.B12 (GNDB2), J1.G1 (GND/SHIELD), J1.G2 (GND/SHIELD), J1.G3 (GND/SHIELD), J1.G4 (GND/SHIELD), J1.S1 (GND/SHIELD), J1.S2 (GND/SHIELD), J1.S3 (GND/SHIELD), J1.S4 (GND/SHIELD), J2.1, R1.2, R10.1, R2.1, R3.1, R4.1, R5.1, R9.2, U1.10 (V_{SS}), U1.11 (V_{SS}), U1.21 (V_{SS}), VR1.1 (GND)
- new net PWR_LED: LED1.1, R10.2
- new net USB_DN: J1.A7 (DN1), J1.B7 (DN2)
- new net USB_DP: J1.A6 (DP1), J1.B6 (DP2)
- new net VBAT: J2.2, U1.14 (V_{BAT}), U1.15 (V_{BAT}), U1.16 (V_{BAT_SENSE})
- new net VBUS: C1.1, F1.2, J1.A4 (VBUSA1), J1.A9 (VBUSA2), J1.B4 (VBUSB1), J1.B9 (VBUSB2)
- no-connect marks 0 -> 12
Other:
- added sheet ESP32_module (ESP32_module.kicad_sch)
- note added: "3.3V Indicator"
- note added: "Battery JST Connector"
- note added: "LiPo Battery Charger"
- note added: "USB-C Connector Circuit"
- note added: "Voltage Regulator"
- title: (none) -> ESP32 Custom Board

Commit message: Completed Schematic Layout
Parts:
- C1: footprint (none) -> Capacitor_SMD:C_0805_2012Metric
- C2: value 0..1uF -> 0.1uF; footprint (none) -> Capacitor_SMD:C_0805_2012Metric
- C3, C5: footprint (none) -> T491A106M016AT:RESC3216X125N
- C7, C8, R1, R10, R2, R3, R4, R5, R6, R7, R8, R9: footprint (none) -> Resistor_SMD:R_0805_2012Metric
- D2: footprint digikey-footprints:0805 -> Resistor_SMD:R_0805_2012Metric
- D3: footprint LTST-C170GKT:LED_LTST-C170GKT -> Resistor_SMD:R_0805_2012Metric
- F1: footprint 0ZCH0110AF2E:FUSC3225X100N -> Resistor_SMD:R_0805_2012Metric
- J1: footprint SS-52400-003:BELFUSE_SS-52400-003 -> Resistor_SMD:R_0805_2012Metric
- J2: footprint B2B-PH-SM4-TB:JST_B2B-PH-SM4-TB -> Resistor_SMD:R_0805_2012Metric
- LED1, LED3: footprint LED_LTST-C170KRKT_LTO -> Resistor_SMD:R_0805_2012Metric
Other:
- moved on the sheet: C1, C2, C3, C7, C8, D2, D3, F1, LED1, LED3, R1, R10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

Commit message: Fixed the Footprint assignment nonsense
Parts:
- C7, C8: footprint Resistor_SMD:R_0805_2012Metric -> Capacitor_SMD:C_0805_2012Metric
- D2: footprint Resistor_SMD:R_0805_2012Metric -> digikey-footprints:0805
- D3: footprint Resistor_SMD:R_0805_2012Metric -> LTST-C170GKT:LED_LTST-C170GKT
- F1: footprint Resistor_SMD:R_0805_2012Metric -> 0ZCH0110AF2E:FUSC3225X100N
- J1: footprint Resistor_SMD:R_0805_2012Metric -> SS-52400-003:BELFUSE_SS-52400-003
- J2: footprint Resistor_SMD:R_0805_2012Metric -> B2B-PH-SM4-TB:JST_B2B-PH-SM4-TB
- LED1, LED3: footprint Resistor_SMD:R_0805_2012Metric -> LTST-C170KRKT:LED_LTST-C170KRKT_LTO
Changed lines of the file:
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@@
 			)
 		)
-		(property "Footprint" "Resistor_SMD:R_0805_2012Metric"
+		(property "Footprint" "digikey-footprints:0805"
 			(at 162.56 48.26 0)
 			(effects
@@
 			)
 		)
+		(property "Purpose" ""
+			(at 167.64 53.34 0)
+			(effects
+				(font
+					(size 1.27 1.27)
+				)
+			)
+		)
 		(pin "1"
 		)
@@
 			)
 		)
-		(property "Footprint" "Resistor_SMD:R_0805_2012Metric"
+		(property "Footprint" "Capacitor_SMD:C_0805_2012Metric"
 			(at 115.2652 132.08 0)
 			(effects
@@
 			)
 		)
-		(property "Footprint" "Resistor_SMD:R_0805_2012Metric"
+		(property "Footprint" "0ZCH0110AF2E:FUSC3225X100N"
 			(at 114.3 45.72 0)
 			(effects
@@
 			)
 		)
-		(property "Footprint" "Resistor_SMD:R_0805_2012Metric"
+		(property "Footprint" "LTST-C170GKT:LED_LTST-C170GKT"
 			(at 177.8 53.34 0)
 			(effects
@@
 			)
 		)
-		(property "Footprint" "Resistor_SMD:R_0805_2012Metric"
+		(property "Footprint" "SS-52400-003:BELFUSE_SS-52400-003"
 			(at 60.96 53.34 0)
 			(effects
@@
 			)
 		)
-		(property "Footprint" "Resistor_SMD:R_0805_2012Metric"
+		(property "Footprint" "Capacitor_SMD:C_0805_2012Metric"
 			(at 33.9852 134.62 0)
 			(effects
@@
 			)
 		)
-		(property "Footprint" "Resistor_SMD:R_0805_2012Metric"
+		(property "Footprint" "LTST-C170KRKT:LED_LTST-C170KRKT_LTO"
 			(at 187.96 63.5 0)
 			(effects
@@
 			)
 		)
-		(property "Footprint" "Resistor_SMD:R_0805_2012Metric"
+		(property "Footprint" "LTST-C170KRKT:LED_LTST-C170KRKT_LTO"
 			(at 233.68 132.08 0)
 			(effects
@@
 			)
 		)
-		(property "Footprint" "Resistor_SMD:R_0805_2012Metric"
+		(property "Footprint" "B2B-PH-SM4-TB:JST_B2B-PH-SM4-TB"
 			(at 60.96 170.18 0)
 			(effects

Commit message: Power copper zones and Placement complete
Parts:
- C8: value 0..1uF -> 0.1uF
Changed lines of the file:
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@@
 	)
 	(rectangle
-		(start 14.224 104.14)
+		(start 14.224 105.156)
 		(end 125.73 149.606)
 		(stroke
@@
 	)
 	(junction
+		(at 93.98 124.46)
+		(diameter 0)
+		(color 0 0 0 0)
+	)
+	(junction
 		(at 256.54 68.58)
 		(diameter 0)
@@
 	(wire
 		(pts
-			(xy 88.9 124.46) (xy 101.6 124.46)
+			(xy 88.9 124.46) (xy 93.98 124.46)
 		)
 		(stroke
@@
 	(wire
 		(pts
+			(xy 93.98 124.46) (xy 101.6 124.46)
+		)
+		(stroke
+			(width 0)
+			(type default)
+		)
+	)
+	(wire
+		(pts
 			(xy 243.84 132.08) (xy 251.46 132.08)
 		)
@@
 		)
 	)
+	(label "+5V"
+		(at 22.86 124.46 180)
+		(effects
+			(font
+				(size 1.27 1.27)
+			)
+			(justify right bottom)
+		)
+	)
 	(label "VBUS"
 		(at 83.82 45.72 0)
@@
 		)
 	)
-	(label "+3.3V"
-		(at 93.98 124.46 90)
-		(effects
-			(font
-				(size 1.27 1.27)
-			)
-			(justify left bottom)
-		)
-	)
 	(label "USB_DP"
 		(at 171.45 128.27 0)
@@
 		)
 	)
-	(label "+3.3V"
-		(at 218.44 121.92 90)
-		(effects
-			(font
-				(size 1.27 1.27)
-			)
-			(justify left bottom)
-		)
-	)
 	(label "VBUS"
 		(at 40.64 58.42 180)
@@
 			)
 		)
-		(property "Value" "0..1uF"
+		(property "Value" "0.1uF"
 			(at 118.11 129.5399 0)
 			(effects
@@
 	)
 	(symbol
+		(lib_id "power:+3.3V")
+		(at 93.98 124.46 0)
+		(unit 1)
+		(exclude_from_sim no)
+		(in_bom yes)
+		(on_board yes)
+		(dnp no)
+		(fields_autoplaced yes)
+		(property "Reference" "#PWR051"
+			(at 93.98 128.27 0)
+			(effects
+				(font
+					(size 1.27 1.27)
+				)
+				(hide yes)
+			)
+		)
+		(property "Value" "+3.3V"
+			(at 93.98 119.38 0)
+			(effects
+				(font
+					(size 1.27 1.27)
+				)
+			)
+		)
+		(property "Footprint" ""
+			(at 93.98 124.46 0)
+			(effects
+				(font
+					(size 1.27 1.27)
+				)
+				(hide yes)
+			)
+		)
+		(property "Datasheet" ""
+			(at 93.98 124.46 0)
+			(effects
+				(font
+					(size 1.27 1.27)
+				)
+				(hide yes)
+			)
+		)
+		(property "Description" "Power symbol creates a global label with name \"+3.3V\""
+			(at 93.98 124.46 0)
+			(effects
+				(font
+					(size 1.27 1.27)
+				)
+				(hide yes)
+			)
+		)
+		(pin "1"
+		)
+		(instances
+			(project ""
+				(path "/8e18a6b6-2497-40ab-aacd-16656297d80d"
+					(reference "#PWR051")
+					(unit 1)
+				)
+			)
+		)
+	)
+	(symbol
 		(lib_id "Battery_Management:MCP73871")
 		(at 220.98 55.88 180)
@@
 	)
 	(symbol
+		(lib_id "power:+3.3V")
+		(at 218.44 121.92 0)
+		(unit 1)
+		(exclude_from_sim no)
+		(in_bom yes)
+		(on_board yes)
+		(dnp no)
+		(fields_autoplaced yes)
+		(property "Reference" "#PWR050"
+			(at 218.44 125.73 0)
+			(effects
+				(font
+					(size 1.27 1.27)
+				)
+				(hide yes)
+			)
+		)
+		(property "Value" "+3.3V"
+			(at 218.44 116.84 0)
+			(effects
+				(font
+					(size 1.27 1.27)
+				)
+			)
+		)
+		(property "Footprint" ""
+			(at 218.44 121.92 0)
+			(effects
+				(font
+					(size 1.27 1.27)
+				)
+				(hide yes)
+			)
+		)
+		(property "Datasheet" ""
+			(at 218.44 121.92 0)
+			(effects
+				(font
+					(size 1.27 1.27)
+				)
+				(hide yes)
+			)
+		)
+		(property "Description" "Power symbol creates a global label with name \"+3.3V\""
+			(at 218.44 121.92 0)
+			(effects
+				(font
+					(size 1.27 1.27)
+				)
+				(hide yes)
+			)
+		)
+		(pin "1"
+		)
+		(instances
+			(project ""
+				(path "/8e18a6b6-2497-40ab-aacd-16656297d80d"
+					(reference "#PWR050")
+					(unit 1)
+				)
+			)
+		)
+	)
+	(symbol
 		(lib_id "0ZCH0110AF2E:0ZCH0110AF2E")
 		(at 114.3 45.72 0)
@@
 					(unit 1)
 				)
-			)
-		)
-	)
-	(symbol
-		(lib_id "power:+5V")
-		(at 22.86 124.46 90)
-		(unit 1)
-		(exclude_from_sim no)
-		(in_bom yes)
-		(on_board yes)
-		(dnp no)
-		(fields_autoplaced yes)
-		(property "Reference" "#PWR011"
-			(at 26.67 124.46 0)
-			(effects
-				(font
-					(size 1.27 1.27)
-				)
-				(hide yes)
-			)
-		)
-		(property "Value" "+5V"
-			(at 19.05 124.4599 90)
-			(effects
-				(font
-					(size 1.27 1.27)
-				)
-				(justify left)
-			)
-		)
-		(property "Footprint" ""
-			(at 22.86 124.46 0)
-			(effects
-				(font
-					(size 1.27 1.27)
-				)
-				(hide yes)
-			)
-		)
-		(property "Datasheet" ""
-			(at 22.86 124.46 0)
-			(effects
-				(font
-					(size 1.27 1.27)
-				)
-				(hide yes)
-			)
-		)
-		(property "Description" "Power symbol creates a global label with name \"+5V\""
-			(at 22.86 124.46 0)
-			(effects
-				(font
-					(size 1.27 1.27)
-				)
-				(hide yes)
-			)
-		)
-		(pin "1"
-		)
-		(instances
-			(project ""
-				(path "/8e18a6b6-2497-40ab-aacd-16656297d80d"
-					(reference "#PWR011")
-					(unit 1)
-				)

Commit message: Completed layout fix
Parts:
- removed D2: LTST-C170TBKT, digikey-footprints:0805, symbol dk_LED-Indication-Discrete:LTST-C170TBKT
- added D2: LTST-C170TBKT, LTST-C170TBKT:DIOC200X125X110, symbol LTST-C170TBKT:LTST-C170TBKT
- added FB1: FBMJ2125HM330-TV, FBMJ2125HM330-TV:BEADC2012X105N, symbol FBMJ2125HM330-TV:FBMJ2125HM330-TV
Connections:
- net +5V: now also FB1.2; no longer U1.1 (OUT), U1.20 (OUT)
- net at R6.1: now also D2.+
- net at U1.7 (STAT2): now also D2.-
- new net: FB1.1, U1.1 (OUT), U1.20 (OUT)
