File: ESP32_module.kicad_sch (KiCad schematic)
At the start: 30 parts, among them J3 GSD090012SEU, U2 CP2102N-Axx-xQFN20, U3 USBLC6-2SC6, U4 W25Q32JVSSIQ, U5 ESP32-C3-WROOM-02-H4

Commit message: Fixed the Footprint assignment nonsense
Parts:
- C10, C11, C12, C13, C14, C6, C9: footprint Resistor_SMD:R_0805_2012Metric -> Capacitor_SMD:C_0805_2012Metric
- D1: footprint Resistor_SMD:R_0805_2012Metric -> CMC-5042PF-AC:CUI_CMC-5042PF-AC
- J3: footprint Resistor_SMD:R_0805_2012Metric -> GSD090012SEU:AMPHENOL_GSD090012SEU
- LED2: footprint Resistor_SMD:R_0805_2012Metric -> LTST-C170KRKT:LED_LTST-C170KRKT_LTO
Changed lines of the file:
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@@
 			)
 		)
-		(property "Footprint" "Resistor_SMD:R_0805_2012Metric"
+		(property "Footprint" "LTST-C170KRKT:LED_LTST-C170KRKT_LTO"
 			(at 119.38 109.22 0)
 			(effects
@@
 			)
 		)
-		(property "Footprint" "Resistor_SMD:R_0805_2012Metric"
+		(property "Footprint" "Capacitor_SMD:C_0805_2012Metric"
 			(at 92.4052 177.8 0)
 			(effects
@@
 			)
 		)
-		(property "Footprint" "Resistor_SMD:R_0805_2012Metric"
+		(property "Footprint" "Capacitor_SMD:C_0805_2012Metric"
 			(at 247.3452 127 0)
 			(effects
@@
 			)
 		)
-		(property "Footprint" "Resistor_SMD:R_0805_2012Metric"
+		(property "Footprint" "Capacitor_SMD:C_0805_2012Metric"
 			(at 71.12 37.1348 0)
 			(effects
@@
 			)
 		)
-		(property "Footprint" "Resistor_SMD:R_0805_2012Metric"
+		(property "Footprint" "Capacitor_SMD:C_0805_2012Metric"
 			(at 257.5052 127 0)
 			(effects
@@
 			)
 		)
-		(property "Footprint" "Resistor_SMD:R_0805_2012Metric"
+		(property "Footprint" "CMC-5042PF-AC:CUI_CMC-5042PF-AC"
 			(at 127 104.14 0)
 			(effects
@@
 			)
 		)
-		(property "Footprint" "Resistor_SMD:R_0805_2012Metric"
+		(property "Footprint" "GSD090012SEU:AMPHENOL_GSD090012SEU"
 			(at 198.12 129.54 0)
 			(effects
@@
 			)
 		)
-		(property "Footprint" "Resistor_SMD:R_0805_2012Metric"
+		(property "Footprint" "Capacitor_SMD:C_0805_2012Metric"
 			(at 260.6548 45.72 0)
 			(effects
@@
 			)
 		)
-		(property "Footprint" "Resistor_SMD:R_0805_2012Metric"
+		(property "Footprint" "Capacitor_SMD:C_0805_2012Metric"
 			(at 272.7452 53.34 0)
 			(effects
@@
 			)
 		)
-		(property "Footprint" "Resistor_SMD:R_0805_2012Metric"
+		(property "Footprint" "Capacitor_SMD:C_0805_2012Metric"
 			(at 71.12 44.7548 0)
 			(effects

Commit message: Fixed ONE MORE Footprint misassignment
Parts:
- D1: footprint CMC-5042PF-AC:CUI_CMC-5042PF-AC -> LTST-C170GKT:LED_LTST-C170GKT
Changed lines of the file:
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@@
 			)
 		)
-		(property "Footprint" "CMC-5042PF-AC:CUI_CMC-5042PF-AC"
+		(property "Footprint" "LTST-C170GKT:LED_LTST-C170GKT"
 			(at 127 104.14 0)
 			(effects

Commit message: Power copper zones and Placement complete
Parts:
- C11, C13: footprint Capacitor_SMD:C_0805_2012Metric -> T491A106M016AT:RESC3216X125N
- C6: footprint Capacitor_SMD:C_0805_2012Metric -> T491A475K016AT:RESC3216X125N
Connections:
- net GND: now also U3.2 (GND); no longer U3.5 (VBUS)
- net USB_DN: now also U3.6 (I/O1); no longer U3.4 (I/O2)
- net USB_DP: now also U3.4 (I/O2); no longer U3.6 (I/O1)
- net VBUS: now also U3.5 (VBUS); no longer U3.2 (GND)
- net USB_N: now reaches U3.1 (I/O1)
- net USB_N: now also U2.5 (D-); no longer U2.4 (D+)
- net USB_P: now reaches U3.3 (I/O2)
- net USB_P: now also U2.4 (D+); no longer U2.5 (D-)
Other:
- moved on the sheet: U3

Commit message: Completed layout fix
Connections:
- net CS_SD: now also U5.4 (IO5); no longer U5.18 (IO0)
- net MIC_OUT: now also U5.18 (IO0); no longer U5.4 (IO5)
Changed lines of the file:
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@@
 	)
 	(junction
-		(at 219.71 116.84)
-		(diameter 0)
-		(color 0 0 0 0)
-	)
-	(junction
 		(at 266.7 55.88)
 		(diameter 0)
@@
 	(wire
 		(pts
+			(xy 91.44 154.94) (xy 91.44 167.64)
+		)
+		(stroke
+			(width 0)
+			(type default)
+		)
+	)
+	(wire
+		(pts
 			(xy 119.38 96.52) (xy 119.38 99.06)
 		)
@@
 	(wire
 		(pts
+			(xy 119.38 124.46) (xy 124.46 124.46)
+		)
+		(stroke
+			(width 0)
+			(type default)
+		)
+	)
+	(wire
+		(pts
 			(xy 251.46 127) (xy 256.54 127)
 		)
@@
 	(wire
 		(pts
-			(xy 91.44 154.94) (xy 91.44 167.64)
-		)
-		(stroke
-			(width 0)
-			(type default)
-		)
-	)
-	(wire
-		(pts
 			(xy 53.34 76.2) (xy 53.34 88.9)
 		)
@@
 	(wire
 		(pts
-			(xy 219.71 116.84) (xy 228.6 116.84)
+			(xy 215.9 116.84) (xy 228.6 116.84)
 		)
 		(stroke
@@
 	(wire
 		(pts
-			(xy 119.38 124.46) (xy 124.46 124.46)
-		)
-		(stroke
-			(width 0)
-			(type default)
-		)
-	)
-	(wire
-		(pts
 			(xy 251.46 127) (xy 251.46 129.54)
 		)
@@
 		)
 	)
-	(wire
-		(pts
-			(xy 215.9 116.84) (xy 219.71 116.84)
-		)
-		(stroke
-			(width 0)
-			(type default)
-		)
-	)
 	(label "MISO_DO"
 		(at 153.67 43.18 0)
@@
 	)
 	(label "CS_SD"
-		(at 193.04 53.34 180)
+		(at 193.04 66.04 180)
 		(effects
 			(font
@@
 	)
 	(label "MIC_OUT"
-		(at 193.04 66.04 180)
+		(at 193.04 53.34 180)
 		(effects
 			(font
@@
 	)
 	(symbol
-		(lib_id "power:+3.3V")
-		(at 76.2 35.56 0)
-		(unit 1)
-		(exclude_from_sim no)
-		(in_bom yes)
-		(on_board yes)
-		(dnp no)
-		(fields_autoplaced yes)
-		(property "Reference" "#PWR011"
-			(at 76.2 39.37 0)
-			(effects
-				(font
-					(size 1.27 1.27)
-				)
-				(hide yes)
-			)
-		)
-		(property "Value" "+3.3V"
-			(at 76.2 30.48 0)
-			(effects
-				(font
-					(size 1.27 1.27)
-				)
-			)
-		)
-		(property "Footprint" ""
-			(at 76.2 35.56 0)
-			(effects
-				(font
-					(size 1.27 1.27)
-				)
-				(hide yes)
-			)
-		)
-		(property "Datasheet" ""
-			(at 76.2 35.56 0)
-			(effects
-				(font
-					(size 1.27 1.27)
-				)
-				(hide yes)
-			)
-		)
-		(property "Description" "Power symbol creates a global label with name \"+3.3V\""
-			(at 76.2 35.56 0)
-			(effects
-				(font
-					(size 1.27 1.27)
-				)
-				(hide yes)
-			)
-		)
-		(pin "1"
-		)
-		(instances
-			(project ""
-				(path "/8e18a6b6-2497-40ab-aacd-16656297d80d/0980fd62-4755-455b-bc26-b8079d26a0ec"
-					(reference "#PWR011")
-					(unit 1)
-				)
-			)
-		)
-	)
-	(symbol
 		(lib_id "LTST-C170KRKT:LTST-C170KRKT")
 		(at 119.38 109.22 90)
@@
 			)
 		)
-		(pin "1"
-		)
-		(instances
-			(project ""
-				(path "/8e18a6b6-2497-40ab-aacd-16656297d80d/0980fd62-4755-455b-bc26-b8079d26a0ec"
-					(reference "#PWR039")
-					(unit 1)
-				)
-			)
-		)
-	)
-	(symbol
-		(lib_id "power:PWR_FLAG")
-		(at 219.71 116.84 0)
-		(unit 1)
-		(exclude_from_sim no)
-		(in_bom yes)
-		(on_board yes)
-		(dnp no)
-		(fields_autoplaced yes)
-		(property "Reference" "#FLG05"
-			(at 219.71 114.935 0)
-			(effects
-				(font
-					(size 1.27 1.27)
-				)
-				(hide yes)
-			)
-		)
-		(property "Value" "PWR_FLAG"
-			(at 219.71 111.76 0)
-			(effects
-				(font
-					(size 1.27 1.27)
-				)
-			)
-		)
-		(property "Footprint" ""
-			(at 219.71 116.84 0)
-			(effects
-				(font
-					(size 1.27 1.27)
-				)
-				(hide yes)
-			)
-		)
-		(property "Datasheet" "~"
-			(at 219.71 116.84 0)
-			(effects
-				(font
-					(size 1.27 1.27)
-				)
-				(hide yes)
-			)
-		)
-		(property "Description" "Special symbol for telling ERC where power comes from"
-			(at 219.71 116.84 0)
+		(property "Purpose" ""
+			(at 238.76 35.56 0)
 			(effects
 				(font
 					(size 1.27 1.27)
 				)
-				(hide yes)
 			)
 		)
@@
 			(project ""
 				(path "/8e18a6b6-2497-40ab-aacd-16656297d80d/0980fd62-4755-455b-bc26-b8079d26a0ec"
-					(reference "#FLG05")
+					(reference "#PWR039")
 					(unit 1)
 				)
@@
 			)
 		)
+		(property "Purpose" ""
+			(at 124.46 127 0)
+			(effects
+				(font
+					(size 1.27 1.27)
+				)
+			)
+		)
 		(pin "1"
 		)
@@
 					(unit 1)
 				)
+			)
+		)
+	)
+	(symbol
+		(lib_id "power:+3.3V")
+		(at 76.2 35.56 0)
+		(unit 1)
+		(exclude_from_sim no)
+		(in_bom yes)
+		(on_board yes)
+		(dnp no)
+		(fields_autoplaced yes)
+		(property "Reference" "#PWR055"
+			(at 76.2 39.37 0)
+			(effects
+				(font
+					(size 1.27 1.27)
+				)
+				(hide yes)
+			)
+		)
+		(property "Value" "+3.3V"
+			(at 76.2 30.48 0)
+			(effects
+				(font
+					(size 1.27 1.27)
+				)
+			)
+		)
+		(property "Footprint" ""
+			(at 76.2 35.56 0)
+			(effects
+				(font
+					(size 1.27 1.27)
+				)
+				(hide yes)
+			)
+		)
+		(property "Datasheet" ""
+			(at 76.2 35.56 0)
+			(effects
+				(font
+					(size 1.27 1.27)
+				)
+				(hide yes)
+			)
+		)
+		(property "Description" "Power symbol creates a global label with name \"+3.3V\""
+			(at 76.2 35.56 0)
+			(effects
+				(font
+					(size 1.27 1.27)
+				)
+				(hide yes)
+			)
+		)
+		(pin "1"
+		)
+		(instances
+			(project ""
+				(path "/8e18a6b6-2497-40ab-aacd-16656297d80d/0980fd62-4755-455b-bc26-b8079d26a0ec"
+					(reference "#PWR055")
+					(unit 1)
+				)
